File: order66/order66.kicad_pcb (KiCad board)
At the start: 2 copper layers, 228.6 x 123 mm, 213 parts, among them J1 NICEVIEW, J2 Pouch Battery Connector, J3 swd connector, J6 millmax connector, SW1 AUX1, SW10 Z, SW100 OFF/ON, SW11 AUX7, SW12 2, SW13 W, SW14 S, SW15 X, SW16 LALT, SW17 3, SW18 E, SW19 D, SW2 ESC, SW20 C, SW21 GUI, SW22 4, SW23 R, SW24 F, SW25 V, SW26 RAISE, SW27 5, SW28 T, SW29 G, SW3 TAB, SW30 B, SW31 LSPACE, SW32 AUX2, SW33 6, SW34 Y, SW35 H, SW36 N, SW37 RSPACE, SW38 AUX3, SW39 7, SW4 CAPSLCK, SW40 U, SW41 J, SW42 M, SW43 LOWER, SW44 AUX4, SW45 8, SW46 I, SW47 K, SW48 ,<, SW49 LEFT, SW5 LSHIFT, SW50 9, SW51 O, SW52 L, SW53 .>, SW54 DOWN, SW55 AUX5, SW56 0, SW57 P, SW58 ;:, SW59 /?, SW6 LCTRL, SW60 UP, SW61 AUX6, SW62 BACKSPACE, SW63 BACKSLASH, SW64 ENTER, SW65 RSHIFT, SW66 RIGHT, SW67 RST, SW68 OFF/ON, SW7 1, SW8 Q, SW9 A, U1 NiceNano

Commit message: 5x12 with backlight wip
Parts:
- removed D121, D122, D123, D124, D125, D126, D127, D128, D129, D130, D131, D132, D133, D134, D135, D136, D137, D138, D139, D140, D141, D142, D143, D144, D145, D146, D147, D148, D149, D150, D151, D152, D153, D154, D155, D156, D157, D158, D159, D160, D161, D162, D163, D164, D165, D166: 1N4148, Diode_SMD:D_SOD-123
- removed J6: millmax connector, Connector_PinHeader_2.54mm:PinHeader_1x02_P2.54mm_Vertical
- removed SW100: OFF/ON, SSSS811101:SW_SSSS811101
- removed SW63: BACKSLASH, MX_Hotswap:MX-Hotswap-1U
- removed SW64: ENTER, MX_Hotswap:MX-Hotswap-1U
- removed SW65: RSHIFT, MX_Hotswap:MX-Hotswap-1U
- removed SW66: RIGHT, MX_Hotswap:MX-Hotswap-1U
- removed SW67: RST, Button_Switch_THT:SW_TH_Tactile_Omron_B3F-10xx
- removed SW68: OFF/ON, footprints:EG1206A_EWI
- added D100: WS2812B, LED_SMD:LED_WS2812B_PLCC4_5.0x5.0mm_P3.2mm, F.Cu at (-177.6, -246.5)
- added D67: WS2812B, LED_SMD:LED_WS2812B_PLCC4_5.0x5.0mm_P3.2mm, F.Cu at (-202.0, -266.4)
- added D68: WS2812B, LED_SMD:LED_WS2812B_PLCC4_5.0x5.0mm_P3.2mm, F.Cu at (-202.0, -259.8)
- added D69: WS2812B, LED_SMD:LED_WS2812B_PLCC4_5.0x5.0mm_P3.2mm, F.Cu at (-202.0, -253.1)
- added D70: WS2812B, LED_SMD:LED_WS2812B_PLCC4_5.0x5.0mm_P3.2mm, F.Cu at (-202.0, -246.5)
- added D71: WS2812B, LED_SMD:LED_WS2812B_PLCC4_5.0x5.0mm_P3.2mm, F.Cu at (-193.9, -306.1)
- added D72: WS2812B, LED_SMD:LED_WS2812B_PLCC4_5.0x5.0mm_P3.2mm, F.Cu at (-193.9, -299.5)
- added D73: WS2812B, LED_SMD:LED_WS2812B_PLCC4_5.0x5.0mm_P3.2mm, F.Cu at (-193.9, -292.9)
- added D74: WS2812B, LED_SMD:LED_WS2812B_PLCC4_5.0x5.0mm_P3.2mm, F.Cu at (-193.9, -286.2)
- added D75: WS2812B, LED_SMD:LED_WS2812B_PLCC4_5.0x5.0mm_P3.2mm, F.Cu at (-193.9, -279.6)
- added D76: WS2812B, LED_SMD:LED_WS2812B_PLCC4_5.0x5.0mm_P3.2mm, F.Cu at (-193.9, -273.0)
- added D77: WS2812B, LED_SMD:LED_WS2812B_PLCC4_5.0x5.0mm_P3.2mm, F.Cu at (-193.9, -266.4)
- added D78: WS2812B, LED_SMD:LED_WS2812B_PLCC4_5.0x5.0mm_P3.2mm, F.Cu at (-193.9, -259.8)
- added D79: WS2812B, LED_SMD:LED_WS2812B_PLCC4_5.0x5.0mm_P3.2mm, F.Cu at (-193.9, -253.1)
- added D80: WS2812B, LED_SMD:LED_WS2812B_PLCC4_5.0x5.0mm_P3.2mm, F.Cu at (-193.9, -246.5)
- added D81: WS2812B, LED_SMD:LED_WS2812B_PLCC4_5.0x5.0mm_P3.2mm, F.Cu at (-185.8, -306.1)
- added D82: WS2812B, LED_SMD:LED_WS2812B_PLCC4_5.0x5.0mm_P3.2mm, F.Cu at (-185.8, -299.5)
- added D83: WS2812B, LED_SMD:LED_WS2812B_PLCC4_5.0x5.0mm_P3.2mm, F.Cu at (-185.8, -292.9)
- added D84: WS2812B, LED_SMD:LED_WS2812B_PLCC4_5.0x5.0mm_P3.2mm, F.Cu at (-185.8, -286.2)
- added D85: WS2812B, LED_SMD:LED_WS2812B_PLCC4_5.0x5.0mm_P3.2mm, F.Cu at (-185.8, -279.6)
- added D86: WS2812B, LED_SMD:LED_WS2812B_PLCC4_5.0x5.0mm_P3.2mm, F.Cu at (-185.8, -273.0)
- added D87: WS2812B, LED_SMD:LED_WS2812B_PLCC4_5.0x5.0mm_P3.2mm, F.Cu at (-185.8, -266.4)
- added D88: WS2812B, LED_SMD:LED_WS2812B_PLCC4_5.0x5.0mm_P3.2mm, F.Cu at (-185.8, -259.8)
- added D89: WS2812B, LED_SMD:LED_WS2812B_PLCC4_5.0x5.0mm_P3.2mm, F.Cu at (-185.8, -253.1)
- added D90: WS2812B, LED_SMD:LED_WS2812B_PLCC4_5.0x5.0mm_P3.2mm, F.Cu at (-185.8, -246.5)
- added D91: WS2812B, LED_SMD:LED_WS2812B_PLCC4_5.0x5.0mm_P3.2mm, F.Cu at (-177.6, -306.1)
- added D92: WS2812B, LED_SMD:LED_WS2812B_PLCC4_5.0x5.0mm_P3.2mm, F.Cu at (-177.6, -299.5)
- added D93: WS2812B, LED_SMD:LED_WS2812B_PLCC4_5.0x5.0mm_P3.2mm, F.Cu at (-177.6, -292.9)
- added D94: WS2812B, LED_SMD:LED_WS2812B_PLCC4_5.0x5.0mm_P3.2mm, F.Cu at (-177.6, -286.2)
- added D95: WS2812B, LED_SMD:LED_WS2812B_PLCC4_5.0x5.0mm_P3.2mm, F.Cu at (-177.6, -279.6)
- added D96: WS2812B, LED_SMD:LED_WS2812B_PLCC4_5.0x5.0mm_P3.2mm, F.Cu at (-177.6, -273.0)
- added D97: WS2812B, LED_SMD:LED_WS2812B_PLCC4_5.0x5.0mm_P3.2mm, F.Cu at (-177.6, -266.4)
- added D98: WS2812B, LED_SMD:LED_WS2812B_PLCC4_5.0x5.0mm_P3.2mm, F.Cu at (-177.6, -259.8)
- added D99: WS2812B, LED_SMD:LED_WS2812B_PLCC4_5.0x5.0mm_P3.2mm, F.Cu at (-177.6, -253.1)
- added J4: millmax connector, Connector_PinHeader_2.54mm:PinHeader_1x02_P2.54mm_Vertical, F.Cu at (-223.3, -198.8)
- BT1: moved to B.Cu
- D1: value 1N4148 -> 1N4148WS; footprint Diode_THT:D_DO-35_SOD27_P7.62mm_Horizontal -> Diode_SMD:D_SOD-323
- D10, D11, D12, D13, D14, D15, D16, D17, D18, D19, D2, D20, D21, D22, D23, D24, D25, D26, D27, D28, D29, D3, D30, D31, D32, D33, D34, D35, D36, D37, D38, D39, D4, D40, D41, D42, D43, D44, D45, D46, D47, D48, D49, D5, D50, D51, D52, D53, D54, D55, D56, D57, D58, D59, D6, D60, D7, D8, D9: value 1N4148 -> 1N4148WS; footprint Diode_THT:D_DO-35_SOD27_P7.62mm_Horizontal -> Diode_SMD:D_SOD-323; moved to F.Cu
- D101, D102, D103, D104, D105, D106, D107, D108, D109, D110, D111, D112, D113, D114, D115, D116, D117, D118, D119, D120: value 1N4148 -> WS2812B; footprint Diode_SMD:D_SOD-123 -> LED_SMD:LED_WS2812B_PLCC4_5.0x5.0mm_P3.2mm; moved to F.Cu
- D61, D62, D63, D64, D65, D66: value 1N4148 -> WS2812B; footprint Diode_THT:D_DO-35_SOD27_P7.62mm_Horizontal -> LED_SMD:LED_WS2812B_PLCC4_5.0x5.0mm_P3.2mm; moved to F.Cu
- J2: moved to F.Cu
- SW1: value AUX1 -> SW_Push
- SW10: value Z -> SW_Push
- SW11: value AUX7 -> SW_Push; moved to F.Cu
- SW12: value 2 -> SW_Push; moved to F.Cu
- SW13: value W -> SW_Push
- SW14: value S -> SW_Push
- SW15: value X -> SW_Push
- SW16: value LALT -> SW_Push
- SW17: value 3 -> SW_Push
- SW18: value E -> SW_Push
- SW19: value D -> SW_Push
- SW2: value ESC -> SW_Push
- SW20: value C -> SW_Push
- SW21: value GUI -> SW_Push
- SW22: value 4 -> SW_Push; moved to F.Cu
- SW23: value R -> SW_Push
- SW24: value F -> SW_Push
- SW25: value V -> SW_Push
- SW26: value RAISE -> SW_Push
- SW27: value 5 -> SW_Push
- SW28: value T -> SW_Push
- SW29: value G -> SW_Push
- SW3: value TAB -> SW_Push
- SW30: value B -> SW_Push
- SW31: value LSPACE -> SW_Push
- SW32: value AUX2 -> SW_Push; moved to F.Cu
- SW33: value 6 -> SW_Push
- SW34: value Y -> SW_Push
- SW35: value H -> SW_Push
- SW36: value N -> SW_Push
- SW37: value RSPACE -> SW_Push
- SW38: value AUX3 -> SW_Push
- SW39: value 7 -> SW_Push
- SW4: value CAPSLCK -> SW_Push
- SW40: value U -> SW_Push
- SW41: value J -> SW_Push
- SW42: value M -> SW_Push; moved to F.Cu
- SW43: value LOWER -> SW_Push; moved to F.Cu
- SW44: value AUX4 -> SW_Push; moved to F.Cu
- SW45: value 8 -> SW_Push; moved to F.Cu
- SW46: value I -> SW_Push; moved to F.Cu
- SW47: value K -> SW_Push; moved to F.Cu
- SW48: value ,< -> SW_Push; moved to F.Cu
- SW49: value LEFT -> SW_Push; moved to F.Cu
- SW5: value LSHIFT -> SW_Push
- SW50: value 9 -> SW_Push; moved to F.Cu
- SW51: value O -> SW_Push; moved to F.Cu
- SW52: value L -> SW_Push; moved to F.Cu
- SW53: value .> -> SW_Push; moved to F.Cu
- SW54: value DOWN -> SW_Push; moved to F.Cu
- SW55: value AUX5 -> SW_Push; moved to F.Cu
- SW56: value 0 -> SW_Push; moved to F.Cu
- SW57: value P -> SW_Push; moved to F.Cu
- SW58: value ;: -> SW_Push; moved to F.Cu
- SW59: value /? -> SW_Push; moved to F.Cu
- SW6: value LCTRL -> SW_Push
- SW60: value UP -> SW_Push; moved to F.Cu
- SW61: value AUX6 -> RST; footprint MX_Hotswap:MX-Hotswap-1U -> Button_Switch_THT:SW_TH_Tactile_Omron_B3F-10xx; moved to F.Cu
- SW62: value BACKSPACE -> OFF/ON; footprint MX_Hotswap:MX-Hotswap-1U -> footprints:EG1206A_EWI; moved to F.Cu
- SW7: value 1 -> SW_Push
- SW8: value Q -> SW_Push
- SW9: value A -> SW_Push
- moved SW37 731.1 mm to (-357.1, -280.7)
- moved SW36 725.5 mm to (-357.1, -290.7)
- moved SW35 720.0 mm to (-357.1, -300.8)
- moved SW34 714.6 mm to (-357.1, -310.8)
- moved SW41 700.8 mm to (-357.1, -240.4)
- moved SW40 696.0 mm to (-357.1, -250.5)
- moved SW26 695.8 mm to (-340.4, -290.7)
- moved SW39 691.3 mm to (-357.1, -260.6)
- moved SW25 689.8 mm to (-340.4, -300.8)
- moved SW38 686.6 mm to (-357.1, -270.6)
- moved D66 684.1 mm to (-202.0, -273.0), turned to 0 degrees
- moved SW24 683.9 mm to (-340.4, -310.8)
- moved SW31 678.1 mm to (-340.4, -240.4)
- moved SW23 678.0 mm to (-340.4, -320.9)
- moved D65 676.0 mm to (-202.0, -279.6), turned to 0 degrees
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Connections:
- D10 pad 1: ROW4 -> ROW0
- D101 pad 1: ROW0 -> GND
- D101 pad 2: Net-(D1-A) -> Net-(D100-DIN)
- D102 pad 1: ROW1 -> GND
- D102 pad 2: Net-(D102-A) -> Net-(D101-DIN)
- D103 pad 1: ROW2 -> GND
- D103 pad 2: Net-(D103-A) -> Net-(D102-DIN)
- D104 pad 1: ROW3 -> GND
- D104 pad 2: Net-(D104-A) -> Net-(D103-DIN)
- D105 pad 1: ROW4 -> GND
- D105 pad 2: Net-(D105-A) -> Net-(D104-DIN)
- D106 pad 1: ROW5 -> GND
- D106 pad 2: Net-(D106-A) -> Net-(D105-DIN)
- D107 pad 1: ROW1 -> GND
- D107 pad 2: Net-(D107-A) -> Net-(D106-DIN)
- D108 pad 1: ROW2 -> GND
- D108 pad 2: Net-(D108-A) -> Net-(D107-DIN)
- D109 pad 1: ROW3 -> GND
- D109 pad 2: Net-(D109-A) -> Net-(D109-DOUT)
- D11 pad 1: ROW5 -> ROW0
- D110 pad 1: ROW4 -> GND
- D110 pad 2: Net-(D10-A) -> Net-(D110-DOUT)
- D111 pad 1: ROW5 -> GND
- D111 pad 2: Net-(D11-A) -> Net-(D111-DOUT)
- D112 pad 1: ROW1 -> GND
- D112 pad 2: Net-(D112-A) -> Net-(D112-DOUT)
- D113 pad 1: ROW2 -> GND
- D113 pad 2: Net-(D113-A) -> Net-(D113-DOUT)
- D114 pad 1: ROW3 -> GND
- D114 pad 2: Net-(D114-A) -> Net-(D114-DOUT)
- D115 pad 1: ROW4 -> GND
- D115 pad 2: Net-(D115-A) -> Net-(D115-DOUT)
- D116 pad 1: ROW5 -> GND
- D116 pad 2: Net-(D116-A) -> Net-(D116-DOUT)
- D117 pad 1: ROW1 -> GND
- D117 pad 2: Net-(D117-A) -> Net-(D117-DOUT)
- D118 pad 1: ROW2 -> GND
- D118 pad 2: Net-(D118-A) -> Net-(D118-DOUT)
- D119 pad 1: ROW3 -> GND
- D119 pad 2: Net-(D119-A) -> Net-(D119-DOUT)
- D12 pad 1: ROW1 -> ROW0
- D12 pad 2: Net-(D112-A) -> Net-(D12-A)
- D120 pad 1: ROW4 -> GND
- D120 pad 2: Net-(D120-A) -> unconnected-(D120-DOUT-Pad2)
- D13 pad 1: ROW2 -> ROW1
- D13 pad 2: Net-(D113-A) -> Net-(D13-A)
- D14 pad 1: ROW3 -> ROW1
- D14 pad 2: Net-(D114-A) -> Net-(D14-A)
- D15 pad 1: ROW4 -> ROW1
- D15 pad 2: Net-(D115-A) -> Net-(D15-A)
- D16 pad 1: ROW5 -> ROW1
- D16 pad 2: Net-(D116-A) -> Net-(D16-A)
- D17 pad 2: Net-(D117-A) -> Net-(D17-A)
- D18 pad 1: ROW2 -> ROW1
- D18 pad 2: Net-(D118-A) -> Net-(D18-A)
- D19 pad 1: ROW3 -> ROW1
- D19 pad 2: Net-(D119-A) -> Net-(D19-A)
- D2 pad 1: ROW1 -> ROW0
- D2 pad 2: Net-(D102-A) -> Net-(D2-A)
- D20 pad 1: ROW4 -> ROW1
- D20 pad 2: Net-(D120-A) -> Net-(D20-A)
- D21 pad 1: ROW5 -> ROW1
- D21 pad 2: Net-(D121-A) -> Net-(D21-A)
- D22 pad 2: Net-(D122-A) -> Net-(D22-A)
- D23 pad 1: ROW2 -> ROW1
- D23 pad 2: Net-(D123-A) -> Net-(D23-A)
- D24 pad 1: ROW3 -> ROW1
- D24 pad 2: Net-(D124-A) -> Net-(D24-A)
- D25 pad 1: ROW4 -> ROW2
- D25 pad 2: Net-(D125-A) -> Net-(D25-A)
- D26 pad 1: ROW5 -> ROW2
- D26 pad 2: Net-(D126-A) -> Net-(D26-A)
- D27 pad 1: ROW1 -> ROW2
- D27 pad 2: Net-(D127-A) -> Net-(D27-A)
- D28 pad 2: Net-(D128-A) -> Net-(D28-A)
- D29 pad 1: ROW3 -> ROW2
- D29 pad 2: Net-(D129-A) -> Net-(D29-A)
- D3 pad 1: ROW2 -> ROW0
- D3 pad 2: Net-(D103-A) -> Net-(D3-A)
- D30 pad 1: ROW4 -> ROW2
- D30 pad 2: Net-(D130-A) -> Net-(D30-A)
- D31 pad 1: ROW5 -> ROW2
- D31 pad 2: Net-(D131-A) -> Net-(D31-A)
- D32 pad 1: ROW0 -> ROW2
- D32 pad 2: Net-(D132-A) -> Net-(D32-A)
- D33 pad 1: ROW1 -> ROW2
- D33 pad 2: Net-(D133-A) -> Net-(D33-A)
- D34 pad 2: Net-(D134-A) -> Net-(D34-A)
- D35 pad 1: ROW3 -> ROW2
- D35 pad 2: Net-(D135-A) -> Net-(D35-A)
- D36 pad 1: ROW4 -> ROW2
- D36 pad 2: Net-(D136-A) -> Net-(D36-A)
- D37 pad 1: ROW5 -> ROW3
- D37 pad 2: Net-(D137-A) -> Net-(D37-A)
- D38 pad 1: ROW0 -> ROW3
- D38 pad 2: Net-(D138-A) -> Net-(D38-A)
- D39 pad 1: ROW1 -> ROW3
- D39 pad 2: Net-(D139-A) -> Net-(D39-A)
- D4 pad 1: ROW3 -> ROW0
- D4 pad 2: Net-(D104-A) -> Net-(D4-A)
- D40 pad 1: ROW2 -> ROW3
- D40 pad 2: Net-(D140-A) -> Net-(D40-A)
- D41 pad 2: Net-(D141-A) -> Net-(D41-A)
- D42 pad 1: ROW4 -> ROW3
- D42 pad 2: Net-(D142-A) -> Net-(D42-A)
- D43 pad 1: ROW5 -> ROW3
- D43 pad 2: Net-(D143-A) -> Net-(D43-A)
- D44 pad 1: ROW0 -> ROW3
- D44 pad 2: Net-(D144-A) -> Net-(D44-A)
- D45 pad 1: ROW1 -> ROW3
- D45 pad 2: Net-(D145-A) -> Net-(D45-A)
- D46 pad 1: ROW2 -> ROW3
- D46 pad 2: Net-(D146-A) -> Net-(D46-A)
- D47 pad 2: Net-(D147-A) -> Net-(D47-A)
- D48 pad 1: ROW4 -> ROW3
- D48 pad 2: Net-(D148-A) -> Net-(D48-A)
- D49 pad 1: ROW5 -> ROW4
- D49 pad 2: Net-(D149-A) -> Net-(D49-A)
- D5 pad 1: ROW4 -> ROW0
- D5 pad 2: Net-(D105-A) -> Net-(D5-A)
- D50 pad 1: ROW1 -> ROW4
- D50 pad 2: Net-(D150-A) -> Net-(D50-A)
- D51 pad 1: ROW2 -> ROW4
- D51 pad 2: Net-(D151-A) -> Net-(D51-A)
- D52 pad 1: ROW3 -> ROW4
- D52 pad 2: Net-(D152-A) -> Net-(D52-A)
- D53 pad 2: Net-(D153-A) -> Net-(D53-A)
- D54 pad 1: ROW5 -> ROW4
- D54 pad 2: Net-(D154-A) -> Net-(D54-A)
- D55 pad 1: ROW0 -> ROW4
- D55 pad 2: Net-(D155-A) -> Net-(D55-A)
- D56 pad 1: ROW1 -> ROW4
- D56 pad 2: Net-(D156-A) -> Net-(D56-A)
- D57 pad 1: ROW2 -> ROW4
- D57 pad 2: Net-(D157-A) -> Net-(D57-A)
- D58 pad 1: ROW3 -> ROW4
- D58 pad 2: Net-(D158-A) -> Net-(D58-A)
- D59 pad 2: Net-(D159-A) -> Net-(D59-A)
- D6 pad 1: ROW5 -> ROW0
- D6 pad 2: Net-(D106-A) -> Net-(D6-A)
- D60 pad 1: ROW5 -> ROW4
- D60 pad 2: Net-(D160-A) -> Net-(D60-A)
- D61 pad 1: ROW0 -> GND
- D61 pad 2: Net-(D161-A) -> Net-(D61-DOUT)
- D62 pad 1: ROW1 -> GND
- D62 pad 2: Net-(D162-A) -> Net-(D62-DOUT)
- D63 pad 1: ROW2 -> GND
- D63 pad 2: Net-(D163-A) -> Net-(D63-DOUT)
- D64 pad 1: ROW3 -> GND
- D64 pad 2: Net-(D164-A) -> Net-(D64-DOUT)
- D65 pad 1: ROW4 -> GND
- D65 pad 2: Net-(D165-A) -> Net-(D65-DOUT)
- D66 pad 1: ROW5 -> GND
- D7 pad 1: ROW1 -> ROW0
- D7 pad 2: Net-(D107-A) -> Net-(D7-A)
- D8 pad 1: ROW2 -> ROW0
- D8 pad 2: Net-(D108-A) -> Net-(D8-A)
- D9 pad 1: ROW3 -> ROW0
- D9 pad 2: Net-(D109-A) -> Net-(D9-A)
- SW1 pad 1: Net-(D1-A) -> COL0
- SW1 pad 2: COL0 -> Net-(D1-A)
- SW10 pad 1: Net-(D10-A) -> COL9
- SW10 pad 2: COL1 -> Net-(D10-A)
- SW11 pad 1: Net-(D11-A) -> COL10
- SW11 pad 2: COL1 -> Net-(D11-A)
- SW12 pad 1: Net-(D112-A) -> COL11
- SW12 pad 2: COL2 -> Net-(D12-A)
- SW13 pad 1: Net-(D113-A) -> COL0
- SW13 pad 2: COL2 -> Net-(D13-A)
- SW14 pad 1: Net-(D114-A) -> COL1
- SW14 pad 2: COL2 -> Net-(D14-A)
- SW15 pad 1: Net-(D115-A) -> COL2
- SW15 pad 2: COL2 -> Net-(D15-A)
- SW16 pad 1: Net-(D116-A) -> COL3
- SW16 pad 2: COL2 -> Net-(D16-A)
- SW17 pad 1: Net-(D117-A) -> COL4
- SW17 pad 2: COL3 -> Net-(D17-A)
- SW18 pad 1: Net-(D118-A) -> COL5
- SW18 pad 2: COL3 -> Net-(D18-A)
- SW19 pad 1: Net-(D119-A) -> COL6
- SW19 pad 2: COL3 -> Net-(D19-A)
- SW2 pad 1: Net-(D102-A) -> COL1
- SW2 pad 2: COL0 -> Net-(D2-A)
- SW20 pad 1: Net-(D120-A) -> COL7
- SW20 pad 2: COL3 -> Net-(D20-A)
- SW21 pad 1: Net-(D121-A) -> COL8
- SW21 pad 2: COL3 -> Net-(D21-A)
- SW22 pad 1: Net-(D122-A) -> COL9
- SW22 pad 2: COL4 -> Net-(D22-A)
- SW23 pad 1: Net-(D123-A) -> COL10
- SW23 pad 2: COL4 -> Net-(D23-A)
- SW24 pad 1: Net-(D124-A) -> COL11
- SW24 pad 2: COL4 -> Net-(D24-A)
- SW25 pad 1: Net-(D125-A) -> COL0
- SW25 pad 2: COL4 -> Net-(D25-A)
- SW26 pad 1: Net-(D126-A) -> COL1
- SW26 pad 2: COL4 -> Net-(D26-A)
- SW27 pad 1: Net-(D127-A) -> COL2
- SW27 pad 2: COL5 -> Net-(D27-A)
- SW28 pad 1: Net-(D128-A) -> COL3
- SW28 pad 2: COL5 -> Net-(D28-A)
- SW29 pad 1: Net-(D129-A) -> COL4
- SW29 pad 2: COL5 -> Net-(D29-A)
- SW3 pad 1: Net-(D103-A) -> COL2
- SW3 pad 2: COL0 -> Net-(D3-A)
- SW30 pad 1: Net-(D130-A) -> COL5
- SW30 pad 2: COL5 -> Net-(D30-A)
- SW31 pad 1: Net-(D131-A) -> COL6
- SW31 pad 2: COL5 -> Net-(D31-A)
- SW32 pad 1: Net-(D132-A) -> COL7
- SW32 pad 2: COL6 -> Net-(D32-A)
- SW33 pad 1: Net-(D133-A) -> COL8
- SW33 pad 2: COL6 -> Net-(D33-A)
- SW34 pad 1: Net-(D134-A) -> COL9
- SW34 pad 2: COL6 -> Net-(D34-A)
- SW35 pad 1: Net-(D135-A) -> COL10
- SW35 pad 2: COL6 -> Net-(D35-A)
- SW36 pad 1: Net-(D136-A) -> COL11
- SW36 pad 2: COL6 -> Net-(D36-A)
- SW37 pad 1: Net-(D137-A) -> COL0
- SW37 pad 2: COL6 -> Net-(D37-A)
- SW38 pad 1: Net-(D138-A) -> COL1
- SW38 pad 2: COL7 -> Net-(D38-A)
- SW39 pad 1: Net-(D139-A) -> COL2
- SW39 pad 2: COL7 -> Net-(D39-A)
- SW4 pad 1: Net-(D104-A) -> COL3
- SW4 pad 2: COL0 -> Net-(D4-A)
- SW40 pad 1: Net-(D140-A) -> COL3
- SW40 pad 2: COL7 -> Net-(D40-A)
- SW41 pad 1: Net-(D141-A) -> COL4
- SW41 pad 2: COL7 -> Net-(D41-A)
- SW42 pad 1: Net-(D142-A) -> COL5
- SW42 pad 2: COL7 -> Net-(D42-A)
- SW43 pad 1: Net-(D143-A) -> COL6
- SW43 pad 2: COL7 -> Net-(D43-A)
- SW44 pad 1: Net-(D144-A) -> COL7
- SW44 pad 2: COL8 -> Net-(D44-A)
- SW45 pad 1: Net-(D145-A) -> COL8
- SW45 pad 2: COL8 -> Net-(D45-A)
- SW46 pad 1: Net-(D146-A) -> COL9
- SW46 pad 2: COL8 -> Net-(D46-A)
- SW47 pad 1: Net-(D147-A) -> COL10
- SW47 pad 2: COL8 -> Net-(D47-A)
- SW48 pad 1: Net-(D148-A) -> COL11
- SW48 pad 2: COL8 -> Net-(D48-A)
- SW49 pad 1: Net-(D149-A) -> COL0
- SW49 pad 2: COL8 -> Net-(D49-A)
- SW5 pad 1: Net-(D105-A) -> COL4
- SW5 pad 2: COL0 -> Net-(D5-A)
- SW50 pad 1: Net-(D150-A) -> COL1
- SW50 pad 2: COL9 -> Net-(D50-A)
- SW51 pad 1: Net-(D151-A) -> COL2
- SW51 pad 2: COL9 -> Net-(D51-A)
- SW52 pad 1: Net-(D152-A) -> COL3
- SW52 pad 2: COL9 -> Net-(D52-A)
- SW53 pad 1: Net-(D153-A) -> COL4
- SW53 pad 2: COL9 -> Net-(D53-A)
- SW54 pad 1: Net-(D154-A) -> COL5
- SW54 pad 2: COL9 -> Net-(D54-A)
- SW55 pad 1: Net-(D155-A) -> COL6
- SW55 pad 2: COL10 -> Net-(D55-A)
- SW56 pad 1: Net-(D156-A) -> COL7
- SW56 pad 2: COL10 -> Net-(D56-A)
- SW57 pad 1: Net-(D157-A) -> COL8
- SW57 pad 2: COL10 -> Net-(D57-A)
- SW58 pad 1: Net-(D158-A) -> COL9
- SW58 pad 2: COL10 -> Net-(D58-A)
- SW59 pad 1: Net-(D159-A) -> COL10
- SW59 pad 2: COL10 -> Net-(D59-A)
- SW6 pad 1: Net-(D106-A) -> COL5
- SW6 pad 2: COL0 -> Net-(D6-A)
- SW60 pad 1: Net-(D160-A) -> COL11
- SW60 pad 2: COL10 -> Net-(D60-A)
- SW61 pad 1: Net-(D161-A) -> RST
- SW61 pad 2: COL11 -> GND
- SW62 pad 1: Net-(D162-A) -> unconnected-(SW62-Pad1)
- SW62 pad 2: COL11 -> BATT+
- SW7 pad 1: Net-(D107-A) -> COL6
- SW7 pad 2: COL1 -> Net-(D7-A)
- SW8 pad 1: Net-(D108-A) -> COL7
- SW8 pad 2: COL1 -> Net-(D8-A)
- SW9 pad 1: Net-(D109-A) -> COL8
- SW9 pad 2: COL1 -> Net-(D9-A)
- U1 pad 7: ROW5 -> BCKLT
Routing:
- net ROW4: track 369.3 -> 0.00 mm
- net ROW3: track 364.4 -> 0.00 mm
- net ROW5: track 355.3 -> 0.00 mm
- net ROW1: track 354.2 -> 0.00 mm
- net ROW2: track 344.0 -> 0.00 mm
- net ROW0: track 290.6 -> 0.00 mm, vias 2 -> 0
- net COL11: track 251.6 -> 0.00 mm, vias 6 -> 0
- net GND: track 231.5 -> 0.00 mm
- net COL10: track 225.8 -> 0.00 mm, vias 6 -> 0
- net COL8: track 193.4 -> 0.00 mm, vias 6 -> 0
- net COL9: track 185.3 -> 0.00 mm, vias 5 -> 0
- net COL7: track 171.2 -> 0.00 mm, vias 6 -> 0
- net COL0: track 154.0 -> 0.00 mm, vias 6 -> 0
- net COL6: track 150.1 -> 0.00 mm, vias 6 -> 0
- net VBATT+: track 140.7 -> 0.00 mm, vias 2 -> 0
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- removed copper zone on B.Cu, net (none)
- removed copper zone on F.Cu, net (none)
Other:
- board size 228.6 x 123 mm -> 107 x 53.1 mm
- board text removed: "order 66"
