File: order66/order66.kicad_pcb (KiCad board)
At the start: 2 copper layers, 107 x 53.1 mm, 194 parts, among them J1 NICEVIEW, J2 Pouch Battery Connector, J3 swd connector, J4 millmax connector, SW1 SW_Push, SW10 SW_Push, SW11 SW_Push, SW12 SW_Push, SW13 SW_Push, SW14 SW_Push, SW15 SW_Push, SW16 SW_Push, SW17 SW_Push, SW18 SW_Push, SW19 SW_Push, SW2 SW_Push, SW20 SW_Push, SW21 SW_Push, SW22 SW_Push, SW23 SW_Push, SW24 SW_Push, SW25 SW_Push, SW26 SW_Push, SW27 SW_Push, SW28 SW_Push, SW29 SW_Push, SW3 SW_Push, SW30 SW_Push, SW31 SW_Push, SW32 SW_Push, SW33 SW_Push, SW34 SW_Push, SW35 SW_Push, SW36 SW_Push, SW37 SW_Push, SW38 SW_Push, SW39 SW_Push, SW4 SW_Push, SW40 SW_Push, SW41 SW_Push, SW42 SW_Push, SW43 SW_Push, SW44 SW_Push, SW45 SW_Push, SW46 SW_Push, SW47 SW_Push, SW48 SW_Push, SW49 SW_Push, SW5 SW_Push, SW50 SW_Push, SW51 SW_Push, SW52 SW_Push, SW53 SW_Push, SW54 SW_Push, SW55 SW_Push, SW56 SW_Push, SW57 SW_Push, SW58 SW_Push, SW59 SW_Push, SW6 SW_Push, SW60 SW_Push, SW61 RST, SW62 OFF/ON, SW7 SW_Push, SW8 SW_Push, SW9 SW_Push, U1 NiceNano

Commit message: wip
Parts:
- D100, D101, D102, D103, D104, D105, D106, D107, D108, D109, D110, D111, D112, D113, D114, D115, D116, D117, D118, D119, D120, D61, D62, D63, D64, D65, D66, D67, D68, D69, D70, D71, D72, D73, D74, D75, D76, D77, D78, D79, D80, D81, D82, D83, D84, D85, D86, D87, D88, D89, D90, D91, D92, D93, D94, D95, D96, D97, D98, D99: footprint LED_SMD:LED_WS2812B_PLCC4_5.0x5.0mm_P3.2mm -> LED_SMD:LED_SK6812MINI_PLCC4_3.5x3.5mm_P1.75mm
- SW11: moved to B.Cu
- SW33: moved to F.Cu
- moved SW21 632.5 mm to (241.8, 43.2)
- moved SW10 584.0 mm to (203.7, 43.2)
- moved SW9 572.5 mm to (184.7, 43.2)
- moved SW8 561.6 mm to (165.6, 43.2)
- moved SW7 551.4 mm to (146.6, 43.2)
- moved SW6 541.8 mm to (127.5, 43.2)
- moved SW5 532.9 mm to (108.5, 43.2)
- moved SW4 524.7 mm to (89.4, 43.2)
- moved SW3 517.3 mm to (70.4, 43.2)
- moved D63 437.0 mm to (70.3, 48.9)
- moved D62 430.7 mm to (51.3, 48.9)
- moved SW33 352.1 mm to (-89.4, -270.6), turned to 0 degrees
- moved SW61 281.1 mm to (-57.1, 19.1)
- moved BT1 251.7 mm to (400.1, 68.7)
- moved SW11 218.5 mm to (222.8, 43.2), turned to 180 degrees
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Other:
- board size 107 x 53.1 mm -> 232.2 x 119.8 mm
